File: L293D/L293D.kicad_pcb (KiCad board)
At the start: 2 copper layers, 60 x 40 mm, 4 parts, among them J1 Screw_Terminal_01x02, J2 Screw_Terminal_01x02, J3 Conn_01x06, U1 L293D

Commit message: pcb
Parts:
- added J4: Screw_Terminal_01x02, TerminalBlock_Phoenix:TerminalBlock_Phoenix_MKDS-1,5-2-5.08_1x02_P5.08mm_Horizontal, F.Cu at (85.4, 78.0)
- moved J1 5.06 mm to (88.0, 60.4), turned to -90 degrees
Connections:
- net Net-(J3-Pin_1) renamed /E34
- J1 pad 1: Net-(J1-Pin_1) -> /1
- J1 pad 2: Net-(J1-Pin_2) -> /2
- J2 pad 1: Net-(J2-Pin_1) -> /3
- J2 pad 2: Net-(J2-Pin_2) -> /4
- J3 pad 2: Net-(J3-Pin_2) -> /4
- J3 pad 3: Net-(J3-Pin_3) -> /3
- J3 pad 4: Net-(J3-Pin_4) -> /2
- J3 pad 5: Net-(J3-Pin_5) -> /1
- J3 pad 6: Net-(J3-Pin_4) -> /E12
- U1 pad 1: Net-(J3-Pin_4) -> /E12
- U1 pad 10: Net-(J3-Pin_3) -> /3
- U1 pad 11: Net-(J2-Pin_1) -> /3
- U1 pad 14: Net-(J2-Pin_2) -> /4
- U1 pad 15: Net-(J3-Pin_2) -> /4
- U1 pad 2: Net-(J3-Pin_5) -> /1
- U1 pad 3: Net-(J1-Pin_1) -> /1
- U1 pad 6: Net-(J1-Pin_2) -> /2
- U1 pad 7: Net-(J3-Pin_4) -> /2
Routing:
- net /1: track 0.00 -> 57.5 mm
- net VCC: track 0.00 -> 53.9 mm
- net /3: track 0.00 -> 52.9 mm
- net GND: track 0.00 -> 49.5 mm
- net /4: track 0.00 -> 45.9 mm
- net Net-(J3-Pin_4): track 43.4 -> 0.00 mm
- net Net-(J3-Pin_5): track 30.3 -> 0.00 mm
- net /2: track 0.00 -> 30.0 mm, vias 0 -> 1
- net /E12: track 0.00 -> 28.5 mm
- net Net-(J3-Pin_2): track 25.0 -> 0.00 mm
- net Net-(J3-Pin_3): track 12.4 -> 0.00 mm
Other:
- board text added: "1 2"
- board text added: "3 4"
- board text added: "E12 1 2 3 4 E34"
- board text added: "Vcc GND"
