File: L293D/L293D.kicad_sch (KiCad schematic)
At the start: 5 parts, among them J1 Screw_Terminal_01x02, J2 Screw_Terminal_01x02, J3 Conn_01x06, J4 Screw_Terminal_01x02, U1 L293D

Commit message: pcb
Connections:
- net 1: now reaches J1.1 (Pin_1), U1.3 (1Y)
- net 1: now also J3.5 (Pin_5), U1.2 (1A)
- net 2: now reaches J1.2 (Pin_2), U1.6 (2Y)
- net 2: now also J3.4 (Pin_4), U1.7 (2A)
- net 3: now reaches J2.1 (Pin_1), U1.11 (3Y)
- net 3: now also J3.3 (Pin_3), U1.10 (3A)
- net 4: now reaches J2.2 (Pin_2), U1.14 (4Y)
- net 4: now also J3.2 (Pin_2), U1.15 (4A)
- net E12: now reaches J3.6 (Pin_6), U1.1 (EN1,2)
- net E12: no longer J3.4 (Pin_4), U1.7 (2A)
- net E34: now reaches J3.1 (Pin_1), U1.9 (EN3,4)
Changed lines of the file:
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@@
 		(color 0 0 0 0)
 	)
-	(junction
-		(at 120.65 80.01)
-		(diameter 0)
-		(color 0 0 0 0)
-	)
-	(wire
-		(pts
-			(xy 120.65 80.01) (xy 120.65 74.93)
+	(wire
+		(pts
+			(xy 120.65 74.93) (xy 120.65 82.55)
 		)
 		(stroke
@@
 	(wire
 		(pts
-			(xy 120.65 82.55) (xy 120.65 80.01)
-		)
-		(stroke
-			(width 0)
-			(type default)
-		)
-	)
-	(wire
-		(pts
 			(xy 175.26 80.01) (xy 175.26 59.69)
 		)
@@
 		)
 	)
+	(label "1"
+		(at 152.4 71.12 0)
+		(fields_autoplaced yes)
+		(effects
+			(font
+				(size 1.27 1.27)
+			)
+			(justify left bottom)
+		)
+	)
+	(label "E34"
+		(at 104.14 90.17 0)
+		(fields_autoplaced yes)
+		(effects
+			(font
+				(size 1.27 1.27)
+			)
+			(justify left bottom)
+		)
+	)
+	(label "4"
+		(at 104.14 87.63 0)
+		(fields_autoplaced yes)
+		(effects
+			(font
+				(size 1.27 1.27)
+			)
+			(justify left bottom)
+		)
+	)
+	(label "E12"
+		(at 104.14 77.47 0)
+		(fields_autoplaced yes)
+		(effects
+			(font
+				(size 1.27 1.27)
+			)
+			(justify left bottom)
+		)
+	)
+	(label "4"
+		(at 152.4 88.9 0)
+		(fields_autoplaced yes)
+		(effects
+			(font
+				(size 1.27 1.27)
+			)
+			(justify left bottom)
+		)
+	)
+	(label "2"
+		(at 152.4 73.66 0)
+		(fields_autoplaced yes)
+		(effects
+			(font
+				(size 1.27 1.27)
+			)
+			(justify left bottom)
+		)
+	)
+	(label "1"
+		(at 104.14 80.01 0)
+		(fields_autoplaced yes)
+		(effects
+			(font
+				(size 1.27 1.27)
+			)
+			(justify left bottom)
+		)
+	)
+	(label "2"
+		(at 104.14 82.55 0)
+		(fields_autoplaced yes)
+		(effects
+			(font
+				(size 1.27 1.27)
+			)
+			(justify left bottom)
+		)
+	)
+	(label "3"
+		(at 152.4 86.36 0)
+		(fields_autoplaced yes)
+		(effects
+			(font
+				(size 1.27 1.27)
+			)
+			(justify left bottom)
+		)
+	)
+	(label "3"
+		(at 104.14 85.09 0)
+		(fields_autoplaced yes)
+		(effects
+			(font
+				(size 1.27 1.27)
+			)
+			(justify left bottom)
+		)
+	)
