File: Relay/Relay.kicad_pcb (KiCad board)
At the start: 2 copper layers, 2 parts, among them J1 Conn_01x04, K1 SRA-12VDC-AL

Commit message: finish
Parts:
- J1: footprint Connector_PinSocket_2.54mm:PinSocket_1x04_P2.54mm_Vertical -> Connector_PinHeader_2.54mm:PinHeader_1x04_P2.54mm_Horizontal
Routing:
- net /sw2: track 0.00 -> 35.2 mm
- net /en-: track 0.00 -> 34.2 mm
- net /en+: track 0.00 -> 27.1 mm
- net /sw1: track 0.00 -> 18.8 mm
Other:
- board outline added: 34.5 x 15 mm
- board text added: "SW1 SW2 EN3 EN4"
