File: Relay/Relay.kicad_sch (KiCad schematic)
At the start: 2 parts, among them J1 Conn_01x04, K1 SRA-12VDC-AL

Commit message: commit PCB
Connections:
- net sw1: now reaches J1.1 (Pin_1), K1.1
- net sw2: now reaches J1.2 (Pin_2), K1.5
- net en-: now reaches J1.3 (Pin_3), K1.3
- net en+: now reaches J1.4 (Pin_4), K1.4
Changed lines of the file:
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@@
+	(wire
+		(pts
+			(xy 147.32 66.04) (xy 147.32 77.47)
+		)
+		(stroke
+			(width 0)
+			(type default)
+		)
+	)
 	(wire
 		(pts
@@
 	(wire
 		(pts
-			(xy 147.32 66.04) (xy 147.32 77.47)
-		)
-		(stroke
-			(width 0)
-			(type default)
-		)
-	)
-	(wire
-		(pts
 			(xy 125.73 74.93) (xy 125.73 76.2)
 		)
@@
 		)
 	)
+	(label "sw2"
+		(at 140.97 74.93 0)
+		(fields_autoplaced yes)
+		(effects
+			(font
+				(size 1.27 1.27)
+			)
+			(justify left bottom)
+		)
+	)
+	(label "en-"
+		(at 147.32 77.47 0)
+		(fields_autoplaced yes)
+		(effects
+			(font
+				(size 1.27 1.27)
+			)
+			(justify left bottom)
+		)
+	)
+	(label "en+"
+		(at 149.86 82.55 0)
+		(fields_autoplaced yes)
+		(effects
+			(font
+				(size 1.27 1.27)
+			)
+			(justify left bottom)
+		)
+	)
+	(label "sw1"
+		(at 141.7447 71.12 0)
+		(fields_autoplaced yes)
+		(effects
+			(font
+				(size 1.27 1.27)
+			)
+			(justify left bottom)
+		)
+	)

Commit message: finish
Parts:
- J1: footprint Connector_PinSocket_2.54mm:PinSocket_1x04_P2.54mm_Vertical -> Connector_PinHeader_2.54mm:PinHeader_1x04_P2.54mm_Horizontal
Changed lines of the file:
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@@
 			)
 		)
-		(property "Footprint" "Connector_PinSocket_2.54mm:PinSocket_1x04_P2.54mm_Vertical"
+		(property "Footprint" "Connector_PinHeader_2.54mm:PinHeader_1x04_P2.54mm_Horizontal"
 			(at 154.94 74.93 0)
 			(effects
