File: ESP8266/ESP8266.kicad_pcb (KiCad board)
At the start: 2 copper layers, 5 parts, among them J1 Conn_01x11, J2 Conn_01x11, SW1 TSC015A03518A, SW2 TSC015A03518A, U1 ESP-12F

Commit message: finish
Parts:
- J1, J2: moved to B.Cu
- moved J1 35.1 mm to (116.0, 40.0), turned to 180 degrees
- moved J2 23.0 mm to (87.0, 65.4)
- moved SW1 4.81 mm to (97.0, 71.0), turned to 90 degrees
- moved SW2 4.81 mm to (105.5, 71.0), turned to 90 degrees
- moved U1 4.08 mm to (101.5, 54.9)
Routing:
- net Net-(J2-Pin_11): track 0.00 -> 31.8 mm, vias 0 -> 2
- net Net-(J1-Pin_8): track 0.00 -> 25.5 mm, vias 0 -> 2
- net Net-(J1-Pin_5): track 0.00 -> 22.5 mm, vias 0 -> 2
- net Net-(J1-Pin_11): track 0.00 -> 14.7 mm
- net Net-(J2-Pin_1): track 0.00 -> 14.6 mm
- net Net-(J2-Pin_2): track 0.00 -> 12.7 mm
- net Net-(J1-Pin_10): track 0.00 -> 12.3 mm
- net Net-(J1-Pin_9): track 0.00 -> 10.5 mm
- net Net-(J2-Pin_3): track 0.00 -> 10.4 mm
- net Net-(J1-Pin_1): track 0.00 -> 10.0 mm
- net Net-(J1-Pin_2): track 0.00 -> 9.55 mm
- net Net-(J2-Pin_10): track 0.00 -> 9.47 mm
- net Net-(J1-Pin_3): track 0.00 -> 9.32 mm
- net Net-(J2-Pin_9): track 0.00 -> 9.24 mm
- net Net-(J1-Pin_4): track 0.00 -> 9.10 mm
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Other:
- board outline added: 34 x 38 mm
